File: Interboard_connector.kicad_sch (KiCad schematic)
At the start: 2 parts, among them J1 Chainbus in, J2 Chainbus Out

Commit message: Done. Don't ask questions
Other:
- title: MMS3 Stepper Controler -> MMS3_hat_protcol_board_basic
Changed lines of the file:
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@@
 	(paper "A4")
 	(title_block
-		(title "MMS3 Stepper Controler")
+		(title "MMS3_hat_protcol_board_basic")
 		(date "2026-02-25")
-		(rev "R0")
+		(rev "A")
 		(company "Moducard System")
 		(comment 1 "Made by Wojciech Szafrański")
