File: MMS3_hat_protcol_board_basic.kicad_sch (KiCad schematic)
At the start: 10 parts

Commit message: Done. Don't ask questions
Parts:
- added C3, C4: 10uF, PCM_JLCPCB:C_0603, symbol PCM_JLCPCB-Capacitors:0603,10uF
- added J11, J4: Conn_01x04_Pin, Connector_JST:JST_XH_S4B-XH-A_1x04_P2.50mm_Horizontal, symbol Connector:Conn_01x04_Pin
- added J7: Conn_01x06_Pin, Connector_JST:JST_XH_S6B-XH-A_1x06_P2.50mm_Horizontal, symbol Connector:Conn_01x06_Pin
- added U3: AMS1117, PCM_JLCPCB:SOT-223-3_L6.5-W3.4-P2.30-LS7.0-BR, symbol PCM_JLCPCB-Power:LDO, 3.3V, 1A
Connections:
- net GND: now also C3.2, C4.2, J11.1 (Pin_1), J4.1 (Pin_1), J7.1 (Pin_1), U3.1 (GND)
- new net +3V3: C4.1, J11.2 (Pin_2), J4.2 (Pin_2), J7.2 (Pin_2), U3.2 (VOUT), U3.4 (VOUT)
- new net +5V: C3.1, U3.3 (VIN)
- new net Chainbus.CS: J7.6 (Pin_6)
- new net Chainbus.MISO: J7.4 (Pin_4)
- new net Chainbus.MOSI: J7.5 (Pin_5)
- new net Chainbus.RX: J11.3 (Pin_3)
- new net Chainbus.SCK: J7.3 (Pin_3)
- new net Chainbus.SCL: J4.4 (Pin_4)
- new net Chainbus.SDA: J4.3 (Pin_3)
- new net Chainbus.TX: J11.4 (Pin_4)
- no-connect marks 2 -> 0
Other:
- removed sheet Buck Regulator
- removed sheet Power Connector
- note added: "3V3 LDO"
- note added: "I2C"
- note added: "LM2596 Step-Down Regulator"
- note added: "SPI"
- note added: "UART"
- title: MMS3 Hat template small (Change Me) -> MMS3_hat_protcol_board_basic
